File: Amplifier_2.sch (KiCad schematic (older format))
At the start: 53 parts, among them U4 BUF602

Commit message: version 1
Parts:
- removed C?: 1u, Capacitors_SMD:C_0603_HandSoldering, symbol C
- removed C?: 30p, Capacitors_SMD:C_0603_HandSoldering, symbol C
- removed C? (x12): 2.2n, Capacitors_SMD:C_0306, symbol C
- removed C? (x3): 2.2u, Capacitors_SMD:C_0402, symbol C
- removed C?: 2.3p, symbol C
- removed C?: 10u, Capacitors_SMD:C_0805_HandSoldering, symbol C
- removed L? (x4): 1k@100MHz, Inductors_SMD:L_1210, symbol Ferrite_Bead_Small
- removed R? (x2): 3.3k, Capacitors_SMD:C_0805_HandSoldering, symbol R
- removed R? (x4): 39, Resistors_SMD:R_0603_HandSoldering, symbol R
- removed R?: 470, Resistors_SMD:R_0603_HandSoldering, symbol R
- removed U? (x2): OPA847, TO_SOT_Packages_SMD:SOT-23-6_Handsoldering, symbol OPA847
- added C100, C101, C92: 2.2u, Capacitors_SMD:C_0402, symbol C
- added C102: 100p, Capacitors_SMD:C_0603_HandSoldering, symbol C
- added C103, C104, C105, C106, C86, C87, C89, C90, C94, C97, C98: 2.2n, Capacitors_SMD:C_0306, symbol C
- added C75: 10u, Capacitors_SMD:C_0805_HandSoldering, symbol C
- added C83: 30p, Capacitors_SMD:C_0603_HandSoldering, symbol C
- added C91: 1u, Capacitors_SMD:C_0603_HandSoldering, symbol C
- added C99: 2.3p, Resistors_SMD:R_0603_HandSoldering, symbol C
- added L16, L17, L18, L19: 1k@100MHz, Inductors_SMD:L_1210, symbol Ferrite_Bead_Small
- added R41, R42, R45, R46: 39, Resistors_SMD:R_0603_HandSoldering, symbol R
- added R43: 470, Resistors_SMD:R_0603_HandSoldering, symbol R
- added R44: 3.3k, Capacitors_SMD:C_0805_HandSoldering, symbol R
- added U20, U22: OPA847, TO_SOT_Packages_SMD:SOT-23-6_Handsoldering, symbol OPA847
- C96: renamed from C?; footprint (none) -> Capacitors_SMD:C_0603_HandSoldering
- gave numbers to parts that had none: 14
- renumbered C13 to C77, C14 to C79, C15 to C81, L6 to L14, R9 to R40, U4 to U19
Connections:
- net AMP_OUT: now also C102.2
- net GND: now also C100.2, C101.2, C103.2, C104.2, C105.2, C106.2, C75.2, C83.2, C86.2, C87.2, C89.2, C91.2, C92.2, C94.2, C97.2, C98.2, R42.2, R45.1, R46.1
- net VCC_-5V: now also L17.2, L19.2
- net buf602_1_V+: now also C92.1, C94.1, C97.1, L18.1
- net buf602_1_V-: now also C98.1, L19.1
- net opa847_0_V+: now also C86.1, L16.1, U20.6 (+V)
- net opa847_0_V-: now also C87.1, C89.1, L17.1, U20.2 (V-)
- net opa847_1_V+: now also C100.1, C103.1, C105.1, U22.6 (+V)
- net opa847_1_V-: now also C101.1, C104.1, C106.1, U22.2 (V-)
- net at U19.1 (out): now also R41.2
- net at U21.4 (In): now also C90.2, R44.1
- net at U21.3 (Ref): now also C91.1, R44.2
- net at R47.1: now also C102.1, C99.1, U22.1 (out)
- net at R47.2: now also C99.2, R45.2, U22.4 (-)
- net at C96.1, U21.1 (out): now also R46.2, U22.3 (+)
- net VCC_+5V renamed VCC_+5V_anlg
- net VCC_+5V_anlg: now also L16.2, L18.2
- new net: R41.1, R43.2, U20.4 (-)
- new net: C90.1, R43.1, U20.1 (out)
- new net: C83.1, R42.1, U20.3 (+)
