File: Discriminator.sch (KiCad schematic (older format))
At the start: 7 parts

Commit message: version 1
Parts:
- removed C? (x3): C, symbol C
- removed R? (x2): R, symbol R
- removed RV?: POT, symbol POT
- removed U?: OP249, symbol OP249
- added C53, C57: 47u, Resistors_SMD:R_0805_HandSoldering, symbol C
- added C54: 100n, Capacitors_SMD:C_0603, symbol C
- added C55, C56, C58, C59, C60, C62, C63: 10u, Resistors_SMD:R_0612, symbol C
- added C61: 100p, Capacitors_SMD:C_0603, symbol C
- added C64: 2.2u, Capacitors_SMD:C_0402_NoSilk, symbol C
- added D3, D4: D, Diodes_SMD:SOD-523, symbol D
- added D5, D6: D_Schottky, Diodes_SMD:D_MiniMELF, symbol D_Schottky
- added R19: 6.8k, Resistors_SMD:R_0805, symbol R
- added R22: 1k, Resistors_SMD:R_0805, symbol R
- added R23: 200, Resistors_SMD:R_0805, symbol R
- added R24, R26: 82.5, Resistors_SMD:R_0603, symbol R
- added R25, R27: 124, Resistors_SMD:R_0603, symbol R
- added RV1: 10k, Potentiometers:Potentiometer_Trimmer_Bourns_3266W, symbol POT
- added RV2: 50k, Potentiometers:Potentiometer_Trimmer_Bourns_3266W, symbol POT
- added U10: ADCMP553, Housings_SSOP:MSOP-8_3x3mm_Pitch0.65mm, symbol ADCMP553
- added U11: MC100ELT21, Housings_SOIC:SOIC-8_3.9x4.9mm_Pitch1.27mm, symbol MC100ELT21
- added U6: TS5A623157, Housings_SSOP:MSOP-10_3x3mm_Pitch0.5mm, symbol TS5A623157
- added U7: MCP6001, TO_SOT_Packages_SMD:SOT-23-5_HandSoldering, symbol MCP6001
- added U8: SN74LVC1G17, TO_SOT_Packages_SMD:SOT-23-5_HandSoldering, symbol SN74LVC1G17
- added U9: MAX9378, Housings_SSOP:TSSOP-8_3x3mm_Pitch0.65mm, symbol MAX9378
Connections:
- net labels added: ADCMP553_+, DISCR_IN, LVDS_OUT_+, LVDS_OUT_-, MCP6001_+, MCP6001_-, PECL_high, PECL_low, TTL_OUT, VCC_+5V_DIG
- net labels removed: Input, Output, VCC_+5V, VCC_-5V
- wire segments 17 -> 74
Other:
- note added: "Remember to check if diode footprint is correct"
