File: Discriminator.sch (KiCad schematic (older format))
At the start: 33 parts, among them U10 ADCMP553, U11 MC100ELT21, U6 TS5A623157, U7 MCP6001, U8 SN74LVC1G17, U9 MAX9378

Commit message: Several bug fixes and improvements.
Parts:
- added C?: 2.2u, Capacitors_SMD:C_0402_NoSilk, symbol C
- added R105: 124, Resistors_SMD:R_0603, symbol R
- added R109: 1k, Resistors_SMD:R_0805, symbol R
- added U31: TC7SZ125FULJ, TO_SOT_Packages_SMD:SOT-353_SC-70-5, symbol TC7SZ125FULJ
Connections:
- net DISCR_IN: now also R105.1; no longer D3.2 (A), D5.1 (K), U10.3 (IN+)
- net GND: now also C?.2, R109.2, U31.1 (~G), U31.3 (GND)
- net TTL_OUT: now also U31.4 (OUT_Y); no longer D6.1 (K), RV2.1, U11.7 (Q)
- net VCC_+5V_DIG: now also C?.1, U31.5 (VCC)
- new net: D3.2 (A), D5.1 (K), R105.2, U10.3 (IN+)
- new net: D6.1 (K), R109.1, RV2.1, U11.7 (Q), U31.2 (IN_A)
Other:
- note removed: "Remember to check if diode footprint is correct"
