File: pmt_driver.sch (KiCad schematic (older format))
At the start: 18 parts

Commit message: version 1
Parts:
- removed J? (x4): Conn_01x02, symbol Conn_01x02
- removed R? (x8): R, symbol R
- removed SW? (x3): SW_DIP_x04, symbol SW_DIP_x04
- removed U? (x3): 74LS153, symbol 74LS153
- added C229, C230: C, Capacitors_SMD:C_0805, symbol C
- added J1, J13, J16, J18, J2: Conn_Coaxial, Connectors:LEMO_angled, symbol Conn_Coaxial
- added J12, J17, J19, J4: Conn_Coaxial, Connectors:LEMO_straight, symbol Conn_Coaxial
- added J24: Conn_01x02, Pin_Headers:Pin_Header_Angled_1x02_Pitch2.54mm, symbol Conn_01x02
- added J3: Jack-DC, Connectors:BARREL_JACK_PJ102B, symbol Jack-DC
- added J5: RJ45, Connectors:RJ45_8_A00-108-262-450, symbol RJ45
- added R1, R20, R61, R71: 50, Resistors_SMD:R_0805, symbol R
Connections:
- net labels added: PECL_H, PECL_L
- net labels removed: +3.3V
- wire segments 131 -> 148
