File: pmt_driver.kicad_pcb (KiCad board)
At the start: 4 copper layers, 249.5 x 160 mm, 2059 parts, among them J1 Conn_Coaxial, J10 Screw_Terminal_01x04, J11 Screw_Terminal_01x04, J12 Conn_Coaxial, J13 Conn_Coaxial, J14 Conn_Coaxial, J15 Conn_Coaxial, J16 Conn_Coaxial, J17 Conn_Coaxial, J18 Conn_Coaxial, J19 Conn_Coaxial, J2 Conn_Coaxial, J20 Conn_Coaxial, J21 Conn_Coaxial, J22 Conn_Coaxial, J23 Conn_Coaxial, J24 Conn_01x02, J3 Jack-DC, J4 Conn_Coaxial, J5 RJ45, J6 Conn_Coaxial, J7 Conn_Coaxial, J8 Screw_Terminal_01x04, J9 Screw_Terminal_01x04, P1 JCH1024D05, P2 PQMC3-D24-S15-S, U1 BB16AH, U10 ADCMP553, U11 MC100ELT21, U12 206-4ST, U13 206-4ST, U14 MAX4634, U15 MAX4634, U16 MAX4634, U17 206-4ST, U18 BUF602, U19 OPA847, U2 BUF602, U20 BUF602, U21 OPA847, U22 BUF602, U23 BUF602, U24 TS5A623157, U25 MCP6001, U26 SN74LVC1G17, U27 MAX9378, U28 ADCMP553, U29 MC100ELT21, U3 OPA847, U30 74HC123A, U31 3310H-001-103L, U32 74HC123A, U33 BUF602, U34 OPA847, U35 BUF602, U36 OPA847, U37 BUF602, U38 BUF602, U39 OPA847, U4 BUF602, U40 BUF602, U41 OPA847, U42 BUF602, U43 TS5A623157, U44 MCP6001, U45 SN74LVC1G17, U46 MAX9378, U47 ADCMP553, U48 MC100ELT21, U49 TS5A623157, U5 OPA847, U50 MCP6001, U51 SN74LVC1G17, U52 MAX9378, U53 ADCMP553, U54 MC100ELT21, U55 DS90LV019, U6 TS5A623157, U7 MCP6001, U8 SN74LVC1G17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

Commit message: v1.1
Parts:
- removed the REF** at (215.4, 99.6)
- removed the REF** at (213.0, 97.6)
- removed the REF** at (139.0, 67.6)
- removed the REF** at (139.4, 45.4)
- removed U31: 3310H-001-103L, Potentiometers:Bourns_3310H
- added C231: 2.2u, Capacitors_SMD:C_0402_NoSilk, F.Cu at (130.5, 113.8)
- added C232: 2.2u, Capacitors_SMD:C_0402_NoSilk, F.Cu at (130.8, 91.8)
- added C233: 2.2u, Capacitors_SMD:C_0402_NoSilk, F.Cu at (130.8, 66.4)
- added C234: 2.2u, Capacitors_SMD:C_0402_NoSilk, F.Cu at (131.2, 44.4)
- added REF**: Via_0.015in, Power_Integrations:Via_0.015in, F.Cu at (129.8, 43.3)
- added REF**: Via_0.015in, Power_Integrations:Via_0.015in, F.Cu at (129.0, 113.8)
- added REF**: Via_0.6mm, Power_Integrations:Via_1mm, F.Cu at (211.8, 95.2)
- added REF**: Via_0.6mm, Power_Integrations:Via_1mm, F.Cu at (211.8, 86.4)
- added REF**: Via_0.015in, Power_Integrations:Via_0.015in, F.Cu at (129.4, 44.4)
- added REF**: Via_0.015in, Power_Integrations:Via_0.015in, F.Cu at (130.8, 43.1)
- added REF**: Via_0.015in, Power_Integrations:Via_0.015in, F.Cu at (129.2, 65.5)
- added REF**: Via_0.015in, Power_Integrations:Via_0.015in, F.Cu at (129.0, 66.4)
- added REF**: Via_0.015in, Power_Integrations:Via_0.015in, F.Cu at (130.2, 65.3)
- added REF**: Via_0.015in, Power_Integrations:Via_0.015in, F.Cu at (129.0, 91.8)
- added REF**: Via_0.015in, Power_Integrations:Via_0.015in, F.Cu at (130.2, 90.6)
- added REF**: Via_0.015in, Power_Integrations:Via_0.015in, F.Cu at (129.0, 112.8)
- added RV14: 10k, Potentiometers:Potentiometer_Trimmer_Bourns_3266W, B.Cu at (203.0, 98.5)
- added RV15: 10k, Potentiometers:Potentiometer_Trimmer_Bourns_3266W, B.Cu at (203.0, 84.3)
- added TP12: TEST, Measurement_Points:Testpoint_Keystone_11011, B.Cu at (232.2, 83.8)
- added TP13: TEST, Measurement_Points:Testpoint_Keystone_11011, B.Cu at (133.8, 116.0)
- added TP15: TEST, Measurement_Points:Testpoint_Keystone_11011, B.Cu at (134.0, 94.0)
- added TP17: TEST, Measurement_Points:Testpoint_Keystone_11011, B.Cu at (134.0, 68.8)
- added TP19: TEST, Measurement_Points:Testpoint_Keystone_11011, B.Cu at (134.5, 46.5)
- added TP5: TEST, Measurement_Points:Testpoint_Keystone_11011, B.Cu at (232.0, 96.5)
- TP1: footprint Measurement_Points:Test_Point_Keystone_5000-5004_Miniature -> Measurement_Points:Testpoint_Keystone_11011; moved to B.Cu
- moved TP7 40.8 mm to (189.5, 90.0)
- moved R22 11.7 mm to (130.2, 116.1)
- moved R82 11.4 mm to (130.8, 68.8)
- moved R50 11.4 mm to (130.8, 94.2)
- moved R89 11.4 mm to (131.2, 46.6)
- moved TP1 11.2 mm to (111.0, 140.2)
- moved REF** 9.96 mm to (129.2, 90.8)
- moved REF** 9.85 mm to (228.2, 133.2)
- moved REF** 9.85 mm to (206.7, 126.4)
- moved REF** 9.85 mm to (209.2, 126.4)
- moved REF** 9.85 mm to (186.2, 126.4)
- moved REF** 9.85 mm to (188.7, 126.4)
- moved C125 9.85 mm to (153.2, 86.0)
- moved C210 9.85 mm to (140.9, 76.2)
- moved C216 9.85 mm to (135.2, 38.8)
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Routing:
- net Net-(C21-Pad1): track 9.88 -> 21.4 mm
- net Net-(C22-Pad1): track 20.0 -> 28.7 mm
- net Net-(JP5-Pad1): track 34.4 -> 26.1 mm
- net Net-(JP5-Pad3): track 51.8 -> 43.4 mm
- net Net-(C233-Pad1): track 2.44 -> 7.57 mm
- net Net-(C232-Pad1): track 2.44 -> 7.54 mm
- net Net-(C234-Pad1): track 2.44 -> 7.49 mm
- net Net-(C231-Pad1): track 2.74 -> 7.54 mm
- net Net-(JP6-Pad3): track 56.9 -> 53.2 mm
- net Net-(JP6-Pad1): track 26.7 -> 23.0 mm
- net Net-(JP7-Pad1): track 85.1 -> 88.3 mm
- net Net-(JP5-Pad2): track 13.3 -> 15.8 mm
- net Net-(JP6-Pad2): track 13.9 -> 16.2 mm
- net Net-(R50-Pad2): track 10.2 -> 9.15 mm
- net Net-(R22-Pad2): track 10.3 -> 9.47 mm
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Other:
- board text added: "+15V"
- board text added: "15V enable"
- board text added: "5.95mV/1µA 1MHz - 300MHz"
- board text added: "50Ω"
- board text added: "CH0"
- board text added: "CH0 (pin 8+ 7-)"
- board text added: "CH0 amp out"
- board text added: "CH0 delay line"
- board text added: "CH1"
- board text added: "CH1 (pin 6+ 5-)"
- board text added: "CH1 amp out"
- board text added: "CH1 delay line"
- board text added: "CH2"
- board text added: "CH2 (pin 4+ 3-)"
- board text added: "CH2 amp out"
- board text added: "CH2 delay line"
- board text added: "CH3"
- board text added: "CH3 (pin 2+ 1-)"
- board text added: "CH3 amp out"
- board text added: "CH3 delay line"
- board text added: "Discriminator"
- board text added: "Gain adjust"
- board text added: "LVDS output"
- board text added: "LVDS trigger"
- board text added: "Monostable multivibrator"
- board text added: "Monostable multivibrators"
- board text added: "Pair A"
- board text added: "Pair B"
- board text added: "Programmable logic (CH0/CH1)"
- board text added: "Programmable logic (CH2/CH3)"
- board text added: "Pulse length adjustment"
- board text added: "TTL trigger"
- board text added: "Trigger length adjustment"
- board text added: "Trigger threshold"
- board text added: "Trigger threshold adjustment"

Commit message: Version 1
Parts:
- removed the REF** at (231.9, 164.8)
- removed the REF** at (231.9, 154.3)
- removed the REF** at (231.9, 149.3)
- added D22: D, Diodes_SMD:DO-214AB_Handsoldering, B.Cu at (230.4, 162.4)
- added REF**: Via_0.6mm, Power_Integrations:Via_1mm, F.Cu at (221.8, 169.8)
- moved REF** 5.99 mm to (234.5, 153.9)
- moved REF** 5.99 mm to (235.5, 152.4)
- moved REF** 5.99 mm to (233.5, 152.4)
- moved REF** 5.99 mm to (231.5, 150.4)
- moved REF** 5.99 mm to (231.5, 148.9)
- moved REF** 5.99 mm to (235.5, 146.9)
- moved REF** 5.99 mm to (238.0, 150.4)
- moved REF** 5.99 mm to (238.0, 148.9)
- moved REF** 5.99 mm to (233.5, 146.9)
- moved D1 5.99 mm to (234.5, 153.3)
Connections:
- F1 pad 1: Net-(C1-Pad1) -> Net-(D22-Pad2)
Routing:
- net Net-(D22-Pad2): track 0.00 -> 4.37 mm
- net Net-(C1-Pad1): track 167.4 -> 171.6 mm
Other:
- board text added: "+"
- board text added: "-"
- board text added: "0"
- board text added: "1"
- board text added: "2"
- board text added: "3"
- board text added: "4"
- board text added: "7"
- board text added: "8"
- board text added: "A"
- board text added: "B"
- board text added: "Magne Eik Lauritzen Nov 01 2017 Rev 1.00"
- board text added: "Monostable circumvent"
- board text added: "OUT"
- board text added: "Pulse output test points"
- board text added: "TRUTH TABLE"
