File: pmt_driver.kicad_pcb (KiCad board)
At the start: 4 copper layers, 249.5 x 160 mm, 2077 parts, among them J1 Conn_Coaxial, J10 Screw_Terminal_01x04, J11 Screw_Terminal_01x04, J12 Conn_Coaxial, J13 Conn_Coaxial, J14 Conn_Coaxial, J15 Conn_Coaxial, J16 Conn_Coaxial, J17 Conn_Coaxial, J18 Conn_Coaxial, J19 Conn_Coaxial, J2 Conn_Coaxial, J20 Conn_Coaxial, J21 Conn_Coaxial, J22 Conn_Coaxial, J23 Conn_Coaxial, J24 Conn_01x02, J3 Jack-DC, J4 Conn_Coaxial, J5 RJ45, J6 Conn_Coaxial, J7 Conn_Coaxial, J8 Screw_Terminal_01x04, J9 Screw_Terminal_01x04, P1 JCH1024D05, P2 PQMC3-D24-S15-S, U1 BB16AH, U10 ADCMP553, U11 MC100ELT21, U12 206-4ST, U13 206-4ST, U14 MAX4634, U15 MAX4634, U16 MAX4634, U17 206-4ST, U18 BUF602, U19 OPA847, U2 BUF602, U20 BUF602, U21 OPA847, U22 BUF602, U23 BUF602, U24 TS5A623157, U25 MCP6001, U26 SN74LVC1G17, U27 MAX9378, U28 ADCMP553, U29 MC100ELT21, U3 OPA847, U30 74HC123A, U32 74HC123A, U33 BUF602, U34 OPA847, U35 BUF602, U36 OPA847, U37 BUF602, U38 BUF602, U39 OPA847, U4 BUF602, U40 BUF602, U41 OPA847, U42 BUF602, U43 TS5A623157, U44 MCP6001, U45 SN74LVC1G17, U46 MAX9378, U47 ADCMP553, U48 MC100ELT21, U49 TS5A623157, U5 OPA847, U50 MCP6001, U51 SN74LVC1G17, U52 MAX9378, U53 ADCMP553, U54 MC100ELT21, U55 DS90LV019, U6 TS5A623157, U7 MCP6001, U8 SN74LVC1G17, U9 MAX9378

Commit message: Several bug fixes and improvements.
Parts:
- removed the REF** at (129.0, 113.8)
- removed the REF** at (58.5, 94.3)
- removed the REF** at (69.1, 94.3)
- removed the REF** at (69.1, 116.3)
- removed the REF** at (58.5, 116.3)
- removed the REF** at (129.4, 44.4)
- removed the REF** at (129.0, 66.4)
- removed the REF** at (129.0, 91.8)
- removed the REF** at (73.6, 41.3)
- removed the REF** at (69.1, 46.9)
- removed the REF** at (69.1, 69.1)
- removed the REF** at (73.6, 63.5)
- added R102: 1k, Resistors_SMD:R_0805, F.Cu at (238.0, 107.8)
- added R103: 1k, Resistors_SMD:R_0805, F.Cu at (238.0, 73.4)
- added R104: 1k, Resistors_SMD:R_0805, F.Cu at (245.0, 81.5)
- added R105: 124, Resistors_SMD:R_0603, F.Cu at (124.2, 111.9)
- added R106: 124, Resistors_SMD:R_0603, F.Cu at (124.2, 89.9)
- added R107: 124, Resistors_SMD:R_0603, F.Cu at (124.5, 64.7)
- added R108: 124, Resistors_SMD:R_0603, F.Cu at (125.0, 42.5)
- added R109: 1k, Resistors_SMD:R_0805, F.Cu at (145.4, 118.4)
- added R110: 1k, Resistors_SMD:R_0805, F.Cu at (145.4, 96.3)
- added R111: 1k, Resistors_SMD:R_0805, F.Cu at (145.8, 71.2)
- added R112: 1k, Resistors_SMD:R_0805, F.Cu at (146.2, 49.1)
- added REF**: Via_0.015in, Power_Integrations:Via_0.015in, F.Cu at (182.7, 60.4)
- added REF**: Via_0.015in, Power_Integrations:Via_0.015in, F.Cu at (244.1, 83.0)
- added REF**: Via_0.015in, Power_Integrations:Via_0.015in, F.Cu at (242.5, 81.4)
- added REF**: Via_0.015in, Power_Integrations:Via_0.015in, F.Cu at (238.9, 109.5)
- added REF**: Via_0.015in, Power_Integrations:Via_0.015in, F.Cu at (238.9, 106.2)
- added REF**: Via_0.015in, Power_Integrations:Via_0.015in, F.Cu at (240.5, 107.8)
- added REF**: Via_0.015in, Power_Integrations:Via_0.015in, F.Cu at (238.9, 75.1)
- added REF**: Via_0.015in, Power_Integrations:Via_0.015in, F.Cu at (240.5, 73.4)
- added REF**: Via_0.015in, Power_Integrations:Via_0.015in, F.Cu at (238.9, 71.8)
- added REF**: Via_0.015in, Power_Integrations:Via_0.015in, F.Cu at (183.4, 61.5)
- added REF**: Via_0.015in, Power_Integrations:Via_0.015in, F.Cu at (182.4, 124.3)
- added REF**: Via_0.015in, Power_Integrations:Via_0.015in, F.Cu at (183.2, 125.5)
- added REF**: Via_0.015in, Power_Integrations:Via_0.015in, F.Cu at (182.2, 109.7)
- added REF**: Via_0.015in, Power_Integrations:Via_0.015in, F.Cu at (183.0, 110.8)
- added REF**: Via_0.015in, Power_Integrations:Via_0.015in, F.Cu at (183.6, 76.1)
- added REF**: Via_0.015in, Power_Integrations:Via_0.015in, F.Cu at (182.8, 75.0)
- added REF**: Via_0.015in, Power_Integrations:Via_0.015in, F.Cu at (244.1, 79.7)
- added U31: TC7SZ125FULJ, TO_SOT_Packages_SMD:SOT-353_SC-70-5, B.Cu at (183.3, 123.0)
- added U56: TC7SZ125FULJ, TO_SOT_Packages_SMD:SOT-353_SC-70-5, B.Cu at (183.2, 108.5)
- added U57: TC7SZ125FULJ, TO_SOT_Packages_SMD:SOT-353_SC-70-5, B.Cu at (183.8, 73.7)
- added U58: TC7SZ125FULJ, TO_SOT_Packages_SMD:SOT-353_SC-70-5, B.Cu at (183.7, 59.1)
- C152, C188, C45, C99: value 2.3p -> 2.2u; footprint Resistors_SMD:R_0603 -> Capacitors_SMD:C_0402_NoSilk
- D1: value D_TVS -> D
- D19, D20, D21: footprint LEDs:LED_D5.0mm -> LEDs:LED_D3.0mm; moved to F.Cu
- R100, R99: value 90 -> 1k
- R101: value 590 -> 4.5k
- R18, R47, R69, R79: value 402 -> 470
- R2: footprint Resistors_SMD:R_0603_HandSoldering -> Resistors_SMD:R_2512
- moved C188 102.6 mm to (184.0, 60.5)
- moved C99 102.5 mm to (183.6, 109.8)
- moved C152 101.8 mm to (184.2, 75.0)
- moved C45 101.5 mm to (183.7, 124.5)
- moved R18 1.04 mm to (83.1, 113.0)
- moved R47 1.04 mm to (83.1, 91.0)
- moved R79 1.04 mm to (83.1, 43.6)
- moved R69 0.99 mm to (83.1, 65.8)
- moved R2 0.95 mm to (96.3, 166.3)
- moved REF** 0.80 mm to (124.2, 90.6)
- moved REF** 0.80 mm to (124.2, 89.2)
- moved REF** 0.62 mm to (134.7, 66.0)
- moved REF** 0.60 mm to (124.2, 112.6)
- moved REF** 0.60 mm to (124.2, 111.2)
- moved REF** 0.45 mm to (124.5, 65.4)
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Connections:
- C152 pad 1: Net-(C152-Pad1) -> +5V
- C152 pad 2: Net-(C152-Pad2) -> GND
- C155 pad 1: Net-(C152-Pad1) -> Net-(C155-Pad1)
- C188 pad 1: Net-(C188-Pad1) -> +5V
- C188 pad 2: Net-(C188-Pad2) -> GND
- C191 pad 1: Net-(C188-Pad1) -> Net-(C191-Pad1)
- C45 pad 1: Net-(C45-Pad1) -> +5V
- C45 pad 2: Net-(C45-Pad2) -> GND
- C48 pad 1: Net-(C45-Pad1) -> Net-(C48-Pad1)
- C99 pad 1: Net-(C102-Pad1) -> +5V
- C99 pad 2: Net-(C99-Pad2) -> GND
- D10 pad 1: /Jumper 2/TTL_IN -> Net-(D10-Pad1)
- D11 pad 2: /Amplifier 3/AMP_OUT -> Net-(D11-Pad2)
- D13 pad 1: /Amplifier 3/AMP_OUT -> Net-(D11-Pad2)
- D14 pad 1: /Jumper 3/TTL_IN -> Net-(D14-Pad1)
- D15 pad 2: /Amplifier 4/AMP_OUT -> Net-(D15-Pad2)
- D17 pad 1: /Amplifier 4/AMP_OUT -> Net-(D15-Pad2)
- D18 pad 1: /Jumper 4/TTL_IN -> Net-(D18-Pad1)
- D3 pad 2: /Amplifier/AMP_OUT -> Net-(D3-Pad2)
- D5 pad 1: /Amplifier/AMP_OUT -> Net-(D3-Pad2)
- D6 pad 1: /Jumper/TTL_IN -> Net-(D6-Pad1)
- D7 pad 2: /Amplifier 2/AMP_OUT -> Net-(D7-Pad2)
- D9 pad 1: /Amplifier 2/AMP_OUT -> Net-(D7-Pad2)
- R16 pad 2: Net-(C45-Pad2) -> Net-(R16-Pad2)
- R18 pad 1: Net-(C45-Pad1) -> Net-(C48-Pad1)
- R18 pad 2: Net-(C45-Pad2) -> Net-(R16-Pad2)
- R45 pad 2: Net-(C99-Pad2) -> Net-(R45-Pad2)
- R47 pad 2: Net-(C99-Pad2) -> Net-(R45-Pad2)
- R67 pad 2: Net-(C152-Pad2) -> Net-(R67-Pad2)
- R69 pad 1: Net-(C152-Pad1) -> Net-(C155-Pad1)
- R69 pad 2: Net-(C152-Pad2) -> Net-(R67-Pad2)
- R77 pad 2: Net-(C188-Pad2) -> Net-(R77-Pad2)
- R79 pad 1: Net-(C188-Pad1) -> Net-(C191-Pad1)
- R79 pad 2: Net-(C188-Pad2) -> Net-(R77-Pad2)
- RV11 pad 1: /Jumper 3/TTL_IN -> Net-(D14-Pad1)
- RV13 pad 1: /Jumper 4/TTL_IN -> Net-(D18-Pad1)
- RV2 pad 1: /Jumper/TTL_IN -> Net-(D6-Pad1)
- RV8 pad 1: /Jumper 2/TTL_IN -> Net-(D10-Pad1)
- U10 pad 3: /Amplifier/AMP_OUT -> Net-(D3-Pad2)
- U11 pad 7: /Jumper/TTL_IN -> Net-(D6-Pad1)
- U21 pad 4: Net-(C99-Pad2) -> Net-(R45-Pad2)
- U28 pad 3: /Amplifier 2/AMP_OUT -> Net-(D7-Pad2)
- U29 pad 7: /Jumper 2/TTL_IN -> Net-(D10-Pad1)
- U36 pad 1: Net-(C152-Pad1) -> Net-(C155-Pad1)
- U36 pad 4: Net-(C152-Pad2) -> Net-(R67-Pad2)
- U41 pad 1: Net-(C188-Pad1) -> Net-(C191-Pad1)
- U41 pad 4: Net-(C188-Pad2) -> Net-(R77-Pad2)
- U47 pad 3: /Amplifier 3/AMP_OUT -> Net-(D11-Pad2)
- U48 pad 7: /Jumper 3/TTL_IN -> Net-(D14-Pad1)
- U5 pad 1: Net-(C45-Pad1) -> Net-(C48-Pad1)
- U5 pad 4: Net-(C45-Pad2) -> Net-(R16-Pad2)
- U53 pad 3: /Amplifier 4/AMP_OUT -> Net-(D15-Pad2)
- U54 pad 7: /Jumper 4/TTL_IN -> Net-(D18-Pad1)
Routing:
- net Net-(D18-Pad1): track 0.00 -> 52.5 mm, vias 0 -> 1
- net Net-(D10-Pad1): track 0.00 -> 52.2 mm, vias 0 -> 1
- net /Jumper 2/TTL_IN: track 67.0 -> 15.3 mm, vias 1 -> 0
- net /Jumper 4/TTL_IN: track 65.6 -> 14.7 mm, vias 1 -> 0
- net /Jumper 3/TTL_IN: track 64.2 -> 14.6 mm, vias 1 -> 0
- net Net-(D14-Pad1): track 0.00 -> 48.8 mm, vias 0 -> 1
- net /Jumper/TTL_IN: track 62.8 -> 15.0 mm, vias 1 -> 0
- net Net-(D6-Pad1): track 0.00 -> 47.7 mm, vias 0 -> 1
- net GND: track 24.5 -> 42.4 mm
- net /Amplifier 2/AMP_OUT: track 41.4 -> 30.3 mm
- net /Amplifier/AMP_OUT: track 41.2 -> 30.2 mm
- net /Amplifier 3/AMP_OUT: track 41.4 -> 30.6 mm
- net /Amplifier 4/AMP_OUT: track 41.8 -> 31.1 mm
- net Net-(D7-Pad2): track 0.00 -> 9.66 mm
- net Net-(D11-Pad2): track 0.00 -> 9.24 mm
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Other:
- board text added: "0,0"
- board text added: "2.950 mm"
- board text added: "4.2mm x 6.55mm"
- board text added: "All measurements in mm. Uncertainty: ±0.1mm"
- board text added: "C"
- board text added: "D"
- board text added: "E"
- board text added: "X : 125.25mm"
- board text added: "X: 190.3 Y: 108.4"
- board text added: "X: 194.1 Y: 71.7"
- board text added: "X: 194.3 Y: 58.9"
- board text added: "X: 196.6 Y: 51.2"
- board text added: "X: 196.6 Y: 79.8"
- board text added: "X: 29.1 Y: 119.8"
- board text added: "X: 57.45 Y: 58.3"
- board text added: "X: 57.45 Y: 72.5"
- board text added: "X: 73.1 Y: 115.5"
- board text added: "X: 82.9 Y: 9.8"
- board text added: "X: 95.85 Y: 91.2"
- board text added: "X: 96.1 Y: 44"
- board text added: "X: 96.1 Y: 69.2"
- board text added: "X: 96.6 Y: 21.75"
- board text added: "Ø:3.2mm"
- board text added: "Ø:5.25mm"
- board text removed: "X:109.2mm Y:30.9mm"
- board text removed: "Ø:5.3mm"

Commit message: Fixed amplifier gain and bandwidth info on silkscreen.
Other:
- board text added: "7.1mV/1µA 1MHz - 370MHz"
- board text removed: "5.95mV/1µA 1MHz - 300MHz"
Changed lines of the file:
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@@
     (34 B.Paste user hide)
     (35 F.Paste user hide)
-    (36 B.SilkS user hide)
-    (37 F.SilkS user)
+    (36 B.SilkS user)
+    (37 F.SilkS user hide)
     (38 B.Mask user hide)
     (39 F.Mask user hide)
@@
   (gr_line (start 63.8 87.1) (end 69.8 91.6) (layer B.SilkS) (width 1))
   (gr_line (start 63.8 91.6) (end 63.8 87.1) (layer B.SilkS) (width 1))
-  (gr_text "5.95mV/1µA\n1MHz - 300MHz" (at 64.3 82.6 180) (layer B.SilkS)
+  (gr_text "7.1mV/1µA\n1MHz - 370MHz" (at 64.3 82.6 180) (layer B.SilkS)
     (effects (font (size 1.5 1.5) (thickness 0.3)) (justify mirror))
   )
@@
   (gr_line (start 130.8 116) (end 133.4 118.4) (layer B.SilkS) (width 1))
   (gr_line (start 130.8 105.6) (end 130.8 116) (layer B.SilkS) (width 1))
-  (gr_text "5.95mV/1µA\n1MHz - 300MHz" (at 64.3 104.2 180) (layer B.SilkS)
+  (gr_text "7.1mV/1µA\n1MHz - 370MHz" (at 64.3 104.2 180) (layer B.SilkS)
     (effects (font (size 1.5 1.5) (thickness 0.3)) (justify mirror))
   )
@@
     (effects (font (size 1.5 1.5) (thickness 0.3)) (justify mirror))
   )
-  (gr_text "5.95mV/1µA\n1MHz - 300MHz" (at 64.3 57.4 180) (layer B.SilkS)
+  (gr_text "7.1mV/1µA\n1MHz - 370MHz" (at 64.3 57.4 180) (layer B.SilkS)
     (effects (font (size 1.5 1.5) (thickness 0.3)) (justify mirror))
   )
@@
   (gr_line (start 131 46.4) (end 133.6 48.8) (layer B.SilkS) (width 1))
   (gr_line (start 131 36) (end 131 46.4) (layer B.SilkS) (width 1))
-  (gr_text "5.95mV/1µA\n1MHz - 300MHz" (at 64.5 35 180) (layer B.SilkS)
+  (gr_text "7.1mV/1µA\n1MHz - 370MHz" (at 64.5 35 180) (layer B.SilkS)
     (effects (font (size 1.5 1.5) (thickness 0.3)) (justify mirror))
   )

Commit message: fixed panel cutout and added custom components and footprints
Other:
- board text removed: "X : 125.25mm"
Changed lines of the file:
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@@
     (area 19.36212 9.6 298.785325 188.25)
     (thickness 1.6)
-    (drawings 836)
+    (drawings 838)
     (tracks 3322)
     (zones 0)
@@
   (page User 297.002 240.005)
   (layers
-    (0 F.Cu power)
-    (1 In1.Cu signal)
-    (2 In2.Cu signal)
-    (31 B.Cu power)
+    (0 F.Cu power hide)
+    (1 In1.Cu signal hide)
+    (2 In2.Cu signal hide)
+    (31 B.Cu power hide)
     (32 B.Adhes user hide)
     (33 F.Adhes user hide)
     (34 B.Paste user hide)
     (35 F.Paste user hide)
-    (36 B.SilkS user)
+    (36 B.SilkS user hide)
     (37 F.SilkS user hide)
     (38 B.Mask user hide)
@@
     (40 Dwgs.User user hide)
     (41 Cmts.User user hide)
-    (42 Eco1.User user hide)
+    (42 Eco1.User user)
     (43 Eco2.User user hide)
     (44 Edge.Cuts user hide)
@@
     (zone_45_only yes)
     (trace_min 0.1524)
-    (segment_width 1)
+    (segment_width 0.3)
     (edge_width 0.1)
     (via_size 0.5334)
@@
     (pad_to_mask_clearance 0.2)
     (aux_axis_origin 37.9 24.8)
-    (visible_elements 7FFECF69)
+    (visible_elements 7FFC0001)
     (pcbplotparams
       (layerselection 0x00400_00000000)
@@
     )
   )
+  (dimension 94.700013 (width 0.3) (layer Eco1.User)
+    (gr_text "94.700 mm" (at 210.54125 30.551751 0.03025120073) (layer Eco1.User)
+      (effects (font (size 1.5 1.5) (thickness 0.3)))
+    )
+    (feature1 (pts (xy 257.9 49.8) (xy 257.891963 29.176751)))
+    (feature2 (pts (xy 163.2 49.85) (xy 163.191963 29.226751)))
+    (crossbar (pts (xy 163.190537 31.926751) (xy 257.890537 31.876751)))
+    (arrow1a (pts (xy 257.890537 31.876751) (xy 256.764343 32.463766)))
+    (arrow1b (pts (xy 257.890537 31.876751) (xy 256.763724 31.290925)))
+    (arrow2a (pts (xy 163.190537 31.926751) (xy 164.31735 32.512577)))
+    (arrow2b (pts (xy 163.190537 31.926751) (xy 164.316731 31.339736)))
+  )
+  (gr_line (start 163.4 72) (end 163.4 54.7) (layer Eco1.User) (width 0.3))
+  (gr_line (start 162.6 119) (end 162.6 101.95) (layer Eco1.User) (width 0.3))
   (gr_line (start 128.5 53.25) (end 124.2 51.55) (layer Eco1.User) (width 0.3))
   (gr_line (start 129.05 55.7) (end 128.5 53.25) (layer Eco1.User) (width 0.3))
@@
     (arrow2b (pts (xy 116.05 118.75) (xy 116.636421 119.876504)))
   )
-  (gr_text "X : 125.25mm" (at 163.2 56.05) (layer Eco1.User)
-    (effects (font (size 1 1) (thickness 0.25)))
-  )
   (gr_text Ø:3.2mm (at 92.35 129) (layer Eco1.User)
