File: power.sch (KiCad schematic (older format))
At the start: 18 parts

Commit message: version 1
Parts:
- removed C? (x9): C, symbol C
- removed L? (x4): L, symbol L
- removed U?: TEN20-2413WIN, Converters_DCDC_ACDC:DCDC-Conv_TRACO_TEN20-xxxx, symbol TEN20-2413WIN
- removed U?: TEN20-2421WIN, Converters_DCDC_ACDC:DCDC-Conv_TRACO_TEN20-xxxx, symbol TEN20-2421WIN
- removed U?: TEN20-2410WIN, Converters_DCDC_ACDC:DCDC-Conv_TRACO_TEN20-xxxx, symbol TEN20-2410WIN
- added C1, C2: 330u, Capacitors_THT:CP_Radial_D10.0mm_P5.00mm, symbol CP
- added C10, C11, C12, C13: 100u, Capacitors_SMD:C_1206_HandSoldering, symbol C
- added C14: 1n, Resistors_SMD:R_1206_HandSoldering, symbol C
- added C16, C17, C18: 10u, Capacitors_SMD:C_0805_HandSoldering, symbol C
- added C19: 12u, Capacitors_THT:C_Radial_D5_L11_P2, symbol CP
- added C20, C4: 100u, Capacitors_THT:CP_Radial_D8.0mm_P3.50mm, symbol CP
- added C3, C5: 4.7u, Capacitors_SMD:C_1206_HandSoldering, symbol C
- added C6, C7, C8, C9: 100u, Capacitors_THT:CP_Radial_D8.0mm_P5.00mm, symbol CP
- added D1: D_TVS, Diodes_SMD:DO-214AB, symbol D_TVS
- added D19, D20, D21: LED, LEDs:LED_D5.0mm, symbol LED
- added D2: D, Diodes_THT:D_DO-41_SOD81_P10.16mm_Horizontal, symbol D
- added F1: Fuse, Fuse_Holders_and_Fuses:Littelfuse_05200101Z_holder, symbol Fuse
- added L1: 56u, Inductors_THT:L_Toroid_Vertical_L22.4mm_W10.2mm_P7.90mm_Vishay_TJ4, symbol L
- added L2: 12u, Inductors_THT:L_Radial_D10.0mm_P5.00mm_Fastron_07M, symbol L
- added L3: 12u, Inductors_THT:L_Radial_D6.0mm_P4.00mm, symbol L
- added L5: 3u, Inductors_THT:L_Radial_D12.0mm_P6.5mm, symbol L
- added P1: JCH1024D05, Modules:JCH1024D05, symbol JCH1024D05
- added P2: PQMC3-D24-S15-S, Modules:PQMC3-S, symbol PQMC3-D24-S15-S
- added R10: 800, Resistors_SMD:R_0805_HandSoldering, symbol R
- added R100, R99: 90, Capacitors_SMD:C_0805, symbol R
- added R101: 590, Capacitors_SMD:C_0805, symbol R
- added R2: 400m, Resistors_SMD:R_0603_HandSoldering, symbol R
- added R3: 300m, Resistors_SMD:R_2010_HandSoldering, symbol R
- added R4: 2.67k, Resistors_SMD:R_0805_HandSoldering, symbol R
- added R5, R6: 180m, Resistors_SMD:R_1206_HandSoldering, symbol R
- added R7: 470, Resistors_SMD:R_0805_HandSoldering, symbol R
- added R8: 910, Resistors_SMD:R_0805_HandSoldering, symbol R
- added R9: 200, Resistors_SMD:R_0805_HandSoldering, symbol R
- added TP10: TEST, symbol TEST
- added U1: BB16AH, Buttons_Switches_THT:BB16AH, symbol BB16AH
- C15: renamed from C?; value C -> 10u; footprint (none) -> Capacitors_SMD:C_0805_HandSoldering; DK (none) -> 399-4925-2-ND; MPN (none) -> C0805C106K8PACTU
- L4: renamed from L?; value L -> 3u; footprint (none) -> Inductors_THT:L_Radial_D12.0mm_P6.5mm; DK (none) -> 732-7146-ND; MPN (none) -> 74475
Connections:
- net labels added: PECL_high, PECL_low
- net labels removed: VCC_3V3, VIN_24V
- wire segments 53 -> 82
Other:
- note removed: "Brick: https://www.digikey.com/product-detail/en/xp-power/VEC40US24/1470-3097-ND/5726817"
- moved on the sheet: C15, L4

Commit message: v1.1
Parts:
- C14: DK 709-1036-6-ND -> 709-1036-1-ND
- TP10: footprint (none) -> Measurement_Points:Test_Point_Keystone_5000-5004_Miniature
Changed lines of the file:
@@
 F 3 "" H 6800 1950 50  0001 C CNN
 F 4 "202R18W102KV4E" H 6800 1950 60  0001 C CNN "MPN"
-F 5 "709-1036-6-ND" H 6800 1950 60  0001 C CNN "DK"
+F 5 "709-1036-1-ND" H 6800 1950 60  0001 C CNN "DK"
 	1    6800 1950
 	0    1    1    0
@@
 F 0 "TP10" H 2200 2250 50  0000 C BNN
 F 1 "TEST" H 2200 2200 50  0000 C CNN
-F 2 "" H 2200 1950 50  0001 C CNN
+F 2 "Measurement_Points:Test_Point_Keystone_5000-5004_Miniature" H 2200 1950 50  0001 C CNN
 F 3 "" H 2200 1950 50  0001 C CNN
 F 4 "36-5001-ND" H 2200 1950 60  0001 C CNN "DK"

Commit message: Version 1
Parts:
- added D22: D, Diodes_SMD:DO-214AB_Handsoldering, symbol D
Connections:
- net at C1.1, D1.1 (A1), R2.2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: now also D22.1 (K); no longer F1.1
- new net: D22.2 (A), F1.1
Other:
- moved on the sheet: D1
Changed lines of the file:
@@
 L D_TVS D1
 U 1 1 59DFEEB0
-P 2350 1350
-F 0 "D1" H 2350 1450 50  0000 C CNN
-F 1 "D_TVS" H 2350 1250 50  0000 C CNN
-F 2 "Diodes_SMD:DO-214AB" H 2350 1350 50  0001 C CNN
-F 3 "" H 2350 1350 50  0001 C CNN
-F 4 "SMCJ48A" H 2350 1350 60  0001 C CNN "MPN"
-F 5 "SMCJ48AFSCT-ND" H 2350 1350 60  0001 C CNN "DK"
-	1    2350 1350
+P 2850 1350
+F 0 "D1" H 2850 1450 50  0000 C CNN
+F 1 "D_TVS" H 2850 1250 50  0000 C CNN
+F 2 "Diodes_SMD:DO-214AB" H 2850 1350 50  0001 C CNN
+F 3 "" H 2850 1350 50  0001 C CNN
+F 4 "SMCJ48A" H 2850 1350 60  0001 C CNN "MPN"
+F 5 "SMCJ48AFSCT-ND" H 2850 1350 60  0001 C CNN "DK"
+	1    2850 1350
 	0    1    1    0
 $EndComp
@@
 $EndComp
 $Comp
-L GND #PWR0115
+L GND #PWR124
 U 1 1 59E06EA6
 P 8750 2800
-F 0 "#PWR0115" H 8750 2550 50  0001 C CNN
+F 0 "#PWR124" H 8750 2550 50  0001 C CNN
 F 1 "GND" H 8750 2650 50  0000 C CNN
 F 2 "" H 8750 2800 50  0001 C CNN
@@
 $EndComp
 $Comp
-L GND #PWR0116
+L GND #PWR121
 U 1 1 59E06F64
 P 5150 3000
-F 0 "#PWR0116" H 5150 2750 50  0001 C CNN
+F 0 "#PWR121" H 5150 2750 50  0001 C CNN
 F 1 "GND" H 5150 2850 50  0000 C CNN
 F 2 "" H 5150 3000 50  0001 C CNN
@@
 GND
 $Comp
-L GND #PWR0117
+L GND #PWR123
 U 1 1 59E0D7E3
 P 7750 2000
-F 0 "#PWR0117" H 7750 1750 50  0001 C CNN
+F 0 "#PWR123" H 7750 1750 50  0001 C CNN
 F 1 "GND" H 7750 1850 50  0000 C CNN
 F 2 "" H 7750 2000 50  0001 C CNN
@@
 $EndComp
 $Comp
-L GND #PWR0118
+L GND #PWR122
 U 1 1 59E16824
 P 7550 4300
-F 0 "#PWR0118" H 7550 4050 50  0001 C CNN
+F 0 "#PWR122" H 7550 4050 50  0001 C CNN
 F 1 "GND" H 7550 4150 50  0000 C CNN
 F 2 "" H 7550 4300 50  0001 C CNN
@@
 	4550 3050 4550 2850
 Wire Wire Line
-	2350 3050 4550 3050
+	2850 3050 4550 3050
 Wire Wire Line
 	4250 2950 4250 3050
 Connection ~ 4250 3050
 Wire Wire Line
-	2150 1200 3150 1200
+	2600 1200 3150 1200
 Wire Wire Line
 	5950 2300 8000 2300
@@
 Wire Wire Line
 	5150 3000 5150 2900
-Connection ~ 2350 1200
+Connection ~ 2850 1200
 Wire Wire Line
 	1700 1200 1850 1200
 Wire Wire Line
-	1700 1500 2350 1500
+	1700 1500 2850 1500
 Wire Wire Line
 	3450 1200 3500 1200
@@
 	3750 2650 3800 2650
 Wire Wire Line
-	2700 2650 3450 2650
+	3100 2650 3450 2650
 Wire Wire Line
 	3300 2950 3300 3050
 Wire Wire Line
-	2350 1500 2350 3050
+	2850 1500 2850 3050
 Connection ~ 3300 2650
 Connection ~ 3300 3050
-Connection ~ 2350 1950
-Wire Wire Line
-	2700 2650 2700 1200
-Connection ~ 2700 1200
+Connection ~ 2850 1950
+Wire Wire Line
+	3100 2650 3100 1200
+Connection ~ 3100 1200
 Wire Wire Line
 	4800 1400 4750 1400
@@
 	1    0    0    -1
 $EndComp
+$Comp
+L D D22
+U 1 1 59F84ACB
+P 2450 1200
+F 0 "D22" H 2450 1300 50  0000 C CNN
+F 1 "D" H 2450 1100 50  0000 C CNN
+F 2 "Diodes_SMD:DO-214AB_Handsoldering" H 2450 1200 50  0001 C CNN
+F 3 "" H 2450 1200 50  0001 C CNN
+F 4 "S3MFSCT-ND" H 2450 1200 60  0001 C CNN "DK"
+F 5 "S3M" H 2450 1200 60  0001 C CNN "MPN"
+	1    2450 1200
+	-1   0    0    1
+$EndComp
+Wire Wire Line
+	2150 1200 2300 1200
 $EndSCHEMATC
