File: power.sch (KiCad schematic (older format))
At the start: 48 parts, among them P1 JCH1024D05, P2 PQMC3-D24-S15-S, U1 BB16AH

Commit message: Several bug fixes and improvements.
Parts:
- removed D1: D_TVS, Diodes_SMD:DO-214AB, symbol D_TVS
- added D1: D, Diodes_SMD:DO-214AB, symbol D
- D19, D20, D21: footprint LEDs:LED_D5.0mm -> LEDs:LED_D3.0mm; DK C503B-GCN-CY0C0791-ND -> 516-3190-1-ND; MPN C503B-GCN-CY0C0791 -> HLMP-1503-C0002
- R100, R99: value 90 -> 1k
- R101: value 590 -> 4.5k
- R2: footprint Resistors_SMD:R_0603_HandSoldering -> Resistors_SMD:R_2512; DK 311-.4QCT-ND -> 311-0.4ARCT-ND; MPN RL0603FR-070R4L -> PT2512FK-070R4L
Connections:
- net GND_RAW: now also D1.2 (A)
- net at C1.1, D22.1 (K), R2.2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: now also D1.1 (K)
Changed lines of the file:
@@
-$EndComp
-$Comp
-L D_TVS D1
-U 1 1 59DFEEB0
-P 2850 1350
-F 0 "D1" H 2850 1450 50  0000 C CNN
-F 1 "D_TVS" H 2850 1250 50  0000 C CNN
-F 2 "Diodes_SMD:DO-214AB" H 2850 1350 50  0001 C CNN
-F 3 "" H 2850 1350 50  0001 C CNN
-F 4 "SMCJ48A" H 2850 1350 60  0001 C CNN "MPN"
-F 5 "SMCJ48AFSCT-ND" H 2850 1350 60  0001 C CNN "DK"
-	1    2850 1350
-	0    1    1    0
 $EndComp
 $Comp
@@
 $EndComp
 $Comp
-L GND #PWR0115
+L GND #PWR0122
 U 1 1 59E06EA6
 P 8750 2800
-F 0 "#PWR0115" H 8750 2550 50  0001 C CNN
+F 0 "#PWR0122" H 8750 2550 50  0001 C CNN
 F 1 "GND" H 8750 2650 50  0000 C CNN
 F 2 "" H 8750 2800 50  0001 C CNN
@@
 $EndComp
 $Comp
-L GND #PWR0116
+L GND #PWR0123
 U 1 1 59E06F64
 P 5150 3000
-F 0 "#PWR0116" H 5150 2750 50  0001 C CNN
+F 0 "#PWR0123" H 5150 2750 50  0001 C CNN
 F 1 "GND" H 5150 2850 50  0000 C CNN
 F 2 "" H 5150 3000 50  0001 C CNN
@@
 F 0 "R2" V 3380 1200 50  0000 C CNN
 F 1 "400m" V 3300 1200 50  0000 C CNN
-F 2 "Resistors_SMD:R_0603_HandSoldering" V 3230 1200 50  0001 C CNN
+F 2 "Resistors_SMD:R_2512" V 3230 1200 50  0001 C CNN
 F 3 "" H 3300 1200 50  0001 C CNN
-F 4 "RL0603FR-070R4L" V 3300 1200 60  0001 C CNN "MPN"
-F 5 "311-.4QCT-ND" V 3300 1200 60  0001 C CNN "DK"
+F 4 "PT2512FK-070R4L" V 3300 1200 60  0001 C CNN "MPN"
+F 5 "311-0.4ARCT-ND" V 3300 1200 60  0001 C CNN "DK"
 	1    3300 1200
 	0    1    1    0
@@
 GND
 $Comp
-L GND #PWR0117
+L GND #PWR0124
 U 1 1 59E0D7E3
 P 7750 2000
-F 0 "#PWR0117" H 7750 1750 50  0001 C CNN
+F 0 "#PWR0124" H 7750 1750 50  0001 C CNN
 F 1 "GND" H 7750 1850 50  0000 C CNN
 F 2 "" H 7750 2000 50  0001 C CNN
@@
 $EndComp
 $Comp
-L GND #PWR0118
+L GND #PWR0125
 U 1 1 59E16824
 P 7550 4300
-F 0 "#PWR0118" H 7550 4050 50  0001 C CNN
+F 0 "#PWR0125" H 7550 4050 50  0001 C CNN
 F 1 "GND" H 7550 4150 50  0000 C CNN
 F 2 "" H 7550 4300 50  0001 C CNN
@@
 F 0 "D19" H 8050 2650 50  0000 C CNN
 F 1 "LED" H 8050 2450 50  0000 C CNN
-F 2 "LEDs:LED_D5.0mm" H 8050 2550 50  0001 C CNN
+F 2 "LEDs:LED_D3.0mm" H 8050 2550 50  0001 C CNN
 F 3 "" H 8050 2550 50  0001 C CNN
-F 4 "C503B-GCN-CY0C0791" H 8050 2550 60  0001 C CNN "MPN"
-F 5 "C503B-GCN-CY0C0791-ND" H 8050 2550 60  0001 C CNN "DK"
+F 4 "HLMP-1503-C0002" H 8050 2550 60  0001 C CNN "MPN"
+F 5 "516-3190-1-ND" H 8050 2550 60  0001 C CNN "DK"
 	1    8050 2550
 	-1   0    0    1
@@
 P 7700 2550
 F 0 "R99" V 7780 2550 50  0000 C CNN
-F 1 "90" V 7700 2550 50  0000 C CNN
+F 1 "1k" V 7700 2550 50  0000 C CNN
 F 2 "Capacitors_SMD:C_0805" V 7630 2550 50  0001 C CNN
 F 3 "" H 7700 2550 50  0001 C CNN
@@
 P 7700 3000
 F 0 "R100" V 7780 3000 50  0000 C CNN
-F 1 "90" V 7700 3000 50  0000 C CNN
+F 1 "1k" V 7700 3000 50  0000 C CNN
 F 2 "Capacitors_SMD:C_0805" V 7630 3000 50  0001 C CNN
 F 3 "" H 7700 3000 50  0001 C CNN
@@
 P 8150 1450
 F 0 "R101" V 8230 1450 50  0000 C CNN
-F 1 "590" V 8150 1450 50  0000 C CNN
+F 1 "4.5k" V 8150 1450 50  0000 C CNN
 F 2 "Capacitors_SMD:C_0805" V 8080 1450 50  0001 C CNN
 F 3 "" H 8150 1450 50  0001 C CNN
@@
 F 0 "D20" H 8050 3100 50  0000 C CNN
 F 1 "LED" H 8050 2900 50  0000 C CNN
-F 2 "LEDs:LED_D5.0mm" H 8050 3000 50  0001 C CNN
+F 2 "LEDs:LED_D3.0mm" H 8050 3000 50  0001 C CNN
 F 3 "" H 8050 3000 50  0001 C CNN
-F 4 "C503B-GCN-CY0C0791" H 8050 3000 60  0001 C CNN "MPN"
-F 5 "C503B-GCN-CY0C0791-ND" H 8050 3000 60  0001 C CNN "DK"
+F 4 "HLMP-1503-C0002" H 8050 3000 60  0001 C CNN "MPN"
+F 5 "516-3190-1-ND" H 8050 3000 60  0001 C CNN "DK"
 	1    8050 3000
 	1    0    0    -1
@@
 F 0 "D21" H 8150 1900 50  0000 C CNN
 F 1 "LED" H 8150 1700 50  0000 C CNN
-F 2 "LEDs:LED_D5.0mm" H 8150 1800 50  0001 C CNN
+F 2 "LEDs:LED_D3.0mm" H 8150 1800 50  0001 C CNN
 F 3 "" H 8150 1800 50  0001 C CNN
-F 4 "C503B-GCN-CY0C0791" H 8150 1800 60  0001 C CNN "MPN"
-F 5 "C503B-GCN-CY0C0791-ND" H 8150 1800 60  0001 C CNN "DK"
+F 4 "HLMP-1503-C0002" H 8150 1800 60  0001 C CNN "MPN"
+F 5 "516-3190-1-ND" H 8150 1800 60  0001 C CNN "DK"
 	1    8150 1800
 	0    -1   -1   0
@@
 Wire Wire Line
 	2150 1200 2300 1200
+$Comp
+L D D1
+U 1 1 5A1CF41D
+P 2850 1350
+F 0 "D1" H 2850 1450 50  0000 C CNN
+F 1 "D" H 2850 1250 50  0000 C CNN
+F 2 "Diodes_SMD:DO-214AB" H 2850 1350 50  0001 C CNN
+F 3 "" H 2850 1350 50  0001 C CNN
+F 4 "SMCJ48AFSCT-ND" H 2850 1350 60  0001 C CNN "DK"
+F 5 "SMCJ48A" H 2850 1350 60  0001 C CNN "MPN"
+	1    2850 1350
+	0    1    1    0
+$EndComp
 $EndSCHEMATC
