File: Amplifier.sch (KiCad schematic (older format))
At the start: 60 parts, among them U2 BUF602, U22 BUF602, U3 OPA847, U4 BUF602, U5 OPA847

Commit message: v1.1
Parts:
- C107, C108, C23, C24, C30, C31, C38, C39, C46, C47: DK 490-14600-1-ND -> 490-10695-1-ND; MPN GRM155R61C225KE11 -> GRM155R61C225KE11DDDD
- R18: DK YAG3125DKR-ND -> YAG3125CT-ND

Commit message: Several bug fixes and improvements.
Parts:
- removed C45: 2.3p, Resistors_SMD:R_0603, symbol C
- C29: DK 399-9057-1-ND -> 490-11324-1-ND; MPN C0603C300J5GACTU -> GRM0335C1H300JA01D
- C42: DK 478-10205-1-ND -> 490-11324-1-ND; MPN 06031A430FAT2A -> GRM0335C1H300JA01D
- R18: value 402 -> 470; DK YAG3125CT-ND -> 311-470LRCT-ND; MPN RC402FR-07402RL -> RC0402FR-07470RL
