File: Logic.sch (KiCad schematic (older format))
At the start: 42 parts, among them U12 206-4ST, U13 206-4ST, U14 MAX4634, U15 MAX4634, U16 MAX4634, U17 206-4ST, U30 74HC123A, U32 74HC123A, U55 DS90LV019

Commit message: Several bug fixes and improvements.
Parts:
- added R102, R103, R104: 1k, Resistors_SMD:R_0805, symbol R
Connections:
- net GND: now also R102.2, R103.2, R104.2
- net at JP7.3, U16.8 (COM), U32.2 (1B): now also R104.1
- net at JP5.3, U14.8 (COM), U30.10 (2B): now also R102.1
- net at JP6.3, U15.8 (COM), U30.2 (1B): now also R103.1
Other:
- moved on the sheet: C75, JP7, R60, RV9, U32A, U55A, U55B
